Commit message: Final version

File: src/ros_gazebo_simulation/description/robot_core.xacro (robot description, xacro)
@@ -78,8 +78,4 @@
         </xacro:inertial_cylinder>
     </link>
-    <!-- <gazebo reference="chassis">
-    <uri>file://media/materials/scripts/gazebo.material</uri>
-        <material>Gazebo\Blue</material>
-    </gazebo> -->
     <!-- LEFT DOWN WHEEL LINK -->
     <joint name="left_down_wheel_joint" type="continuous">
@@ -105,8 +101,4 @@
         </xacro:inertial_cylinder>
     </link>
-    <!-- <gazebo reference="left_down_wheel">
-    <uri>file://media/materials/scripts/gazebo.material</uri>
-        <material>Gazebo\black2</material>
-    </gazebo> -->
     <!-- RIGHT DOWN WHEEL LINK -->
     <joint name="right_down_wheel_joint" type="continuous">
@@ -132,8 +124,4 @@
         </xacro:inertial_cylinder>
     </link>
-    <!-- <gazebo reference="right_down_wheel">
-    <uri>file://media/materials/scripts/gazebo.material</uri>
-        <material>Gazebo\black2</material>
-    </gazebo> -->
     <!-- LEFT UP WHEEL LINK -->
     <joint name="left_up_wheel_joint" type="continuous">
@@ -159,8 +147,4 @@
         </xacro:inertial_cylinder>
     </link>
-    <!-- <gazebo reference="left_up_wheel">
-    <uri>file://media/materials/scripts/gazebo.material</uri>
-        <material>Gazebo\black2</material>
-    </gazebo> -->
     <!-- RIGHT UP WHEEL LINK -->
     <joint name="right_up_wheel_joint" type="continuous">
@@ -186,7 +170,3 @@
         </xacro:inertial_cylinder>
     </link>
-    <!-- <gazebo reference="right_up_wheel">
-        <uri>file://media/materials/scripts/gazebo.material</uri>
-        <material>Gazebo\black2</material>
-    </gazebo> -->
 </robot>
